Commit message: world link fix

File: urdf/panda_arm_generic.urdf.xacro (robot description, xacro)
@@ -10,4 +10,5 @@
   <xacro:arg name="control_mode" default="effort" />
   <xacro:include filename="$(find panda)/urdf/panda_arm_generic.xacro"/>
+  <link name="world"/>
   <xacro:panda_arm_generic  x="$(arg x)"
                             y="$(arg y)"
