Commit message: Better friction parameters, gripper effort controller by default in sim

File: urdf/panda.gazebo.xacro (robot description, xacro)
@@ -12,6 +12,52 @@
             <gazebo reference="${link}">
                 <material>Gazebo/Grey</material>
-                <mu1>0.2</mu1>
-                <mu2>0.2</mu2>
+                <!-- I directly write the sdf specification, it will be merged in the link with the urdf by gazebo
+                     see: http://gazebosim.org/tutorials/?tut=ros_urdf
+                          http://sdformat.org/spec?ver=1.7&elem=collision#link_collision -->
+                <!--
+                <collision>
+                    <surface>
+                        <contact>
+                            <ode>
+                            <kp>1e+06</kp>
+                            <kd>100000</kd>
+                            </ode>
+                        </contact>
+                        <friction>
+                            <ode>
+                            <mu>150</mu>
+                            <mu2>150</mu2>
+                            </ode>
+                        </friction>
+                    </surface>
+                </collision>
+                -->
+                <collision>
+                    <surface>
+                        <contact>
+                            <ode>
+                                <kp>2e+05</kp>
+                                <kd>80</kd>
+                                <!-- Equivalent to CFM = 10e-2, ERP = 0.2, with step size = 10^-3,
+                                    See http://www.ode.org/ode-latest-userguide.html#sec_3_8_2 -->
+                            </ode>
+                        </contact>
+                        <friction>
+                            <torsional>
+                                <coefficient>0.5</coefficient>
+                            </torsional>
+                            <ode>
+                                <!-- Some Coulomb friction coefficient examples:
+                                    https://web.mit.edu/8.13/8.13c/references-fall/aip/aip-handbook-section2d.pdf
+                                    https://engineeringlibrary.org/reference/coefficient-of-friction
+                                    https://www.engineeringtoolbox.com/friction-coefficients-d_778.html
+                                    https://www.tribonet.org/wiki/friction-coefficients-in-atmosphere-and-vacuum/
+                                -->
+                                <mu>0.5</mu>
+                                <mu2>0.5</mu2>
+                            </ode>
+                        </friction>
+                    </surface>
+                </collision>
             </gazebo>
         </xacro:macro>

File: urdf/standard_gripper.xacro (robot description, xacro)
@@ -46,8 +46,4 @@
         <inertia ixx="0.1" ixy="0.0" ixz="0.0" iyy="0.1" iyz="0.0" izz="0.1" />
       </inertial>
-      <gazebo reference="${ns}_leftfinger">
-        <mu1 value="100"/>
-        <mu2 value="100"/>
-      </gazebo>
       <!-- end for simulation -->
     </link>
@@ -71,10 +67,6 @@
         <inertia ixx="0.1" ixy="0.0" ixz="0.0" iyy="0.1" iyz="0.0" izz="0.1" />
       </inertial>
-      <gazebo reference="${ns}_rightfinger">
-        <mu1 value="100"/>
-        <mu2 value="100"/>
-      </gazebo>
       <!-- end for simulation -->
-   </link>
+    </link>
     <joint name="${ns}_finger_joint1" type="prismatic">
       <parent link="${ns}_hand"/>
