Commit message: Use gripper visual meshes for collision

File: urdf/standard_gripper.xacro (robot description, xacro)
@@ -18,5 +18,5 @@
       <collision>
         <geometry>
-          <mesh filename="package://franka_description/meshes/collision/hand.stl"/>
+          <mesh filename="package://franka_description/meshes/visual/hand.dae"/>
         </geometry>
       </collision>
@@ -35,4 +35,9 @@
         </geometry>
       </visual>
+      <collision>
+        <geometry>
+          <mesh filename="package://franka_description/meshes/visual/finger.dae"/>
+        </geometry>
+      </collision>
       <!-- for simulation -->
       <inertial>
@@ -41,4 +46,8 @@
         <inertia ixx="0.1" ixy="0.0" ixz="0.0" iyy="0.1" iyz="0.0" izz="0.1" />
       </inertial>
+      <gazebo reference="${ns}_leftfinger">
+        <mu1 value="100"/>
+        <mu2 value="100"/>
+      </gazebo>
       <!-- end for simulation -->
     </link>
@@ -50,4 +59,10 @@
         </geometry>
       </visual>
+      <collision>
+        <origin xyz="0 0 0" rpy="0 0 ${pi}"/>
+        <geometry>
+          <mesh filename="package://franka_description/meshes/visual/finger.dae"/>
+        </geometry>
+      </collision>
       <!-- for simulation -->
       <inertial>
@@ -56,4 +71,8 @@
         <inertia ixx="0.1" ixy="0.0" ixz="0.0" iyy="0.1" iyz="0.0" izz="0.1" />
       </inertial>
+      <gazebo reference="${ns}_rightfinger">
+        <mu1 value="100"/>
+        <mu2 value="100"/>
+      </gazebo>
       <!-- end for simulation -->
    </link>

Commit message: added tcp link in gripper

File: urdf/standard_gripper.xacro (robot description, xacro)
@@ -84,4 +84,10 @@
       <mimic joint="${ns}_finger_joint1" />
     </joint>
+    <link name="${ns}_tcp"/>
+    <joint name="${ns}_tcp_joint" type="fixed">
+      <parent link="${ns}_hand"/>
+      <child link="${ns}_tcp"/>
+      <origin xyz="0 0 0.1035" rpy="0 0 0"/>
+    </joint>
   </xacro:macro>
 </robot>
